File: Frankenball Orbit.kicad_sch (KiCad schematic)
At the start: 18 parts, among them J101 ADNS-5050, J102 Conn_01x05_Male, J103 Conn_02x04_Odd_Even, Q101 PT2559B, Q102 2N7002, SW101 SW_Push, SW102 SW_Push, U101 74HC14

Commit message: Routing finished
Connections:
- net USB_GND is gone; now on net GND: C101.2, C102.2, J102.3 (Pin_3), R105.2
- net PB12 renamed PBu12
- net PB13 renamed PBu13
- net PB15 renamed PBu15
- net PC1 renamed PB7
- net PC2 renamed PB6
- net PC3 renamed PB5
- net PC4 renamed PB4
- net PC5 renamed PB3
Other:
- removed sheet STM32F401
- added sheet STM32F411 (kicad-hierarchical-blocks/MCUs/STM32F411CCU/STM32F411CCU.kicad_sch)
- moved on the sheet: C101, C102, J102, J103, R105, R106, R107
