File: Frankenball Orbit.kicad_pcb (KiCad board)
At the start: 2 copper layers, 91.9 x 57.4 mm, 45 parts, among them J1 Conn_02x03_Odd_Even, J101 ADNS-5050, J102 Conn_01x05_Male, J103 Conn_02x04_Odd_Even, J2 Conn_02x04_Odd_Even, Q101 PT2559B, Q102 2N7002, SW1 SW_Push, SW101 SW_Push, SW102 SW_Push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

Commit message: Routing finished
Parts:
- removed C15: 100nF, Capacitor_SMD:C_0402_1005Metric
- C1: value 10µF -> 1µF
- C2: value 10µF -> 1µF; footprint Capacitor_Tantalum_SMD:CP_EIA-3216-10_Kemet-I -> Capacitor_SMD:C_0402_1005Metric
- C3: value 10µF -> 100nF; footprint Capacitor_Tantalum_SMD:CP_EIA-3216-10_Kemet-I -> Capacitor_SMD:C_0402_1005Metric
- J2: value Conn_02x04_Odd_Even -> Connector_Generic:Conn_01x05; footprint Connector_PinHeader_2.54mm:PinHeader_2x04_P2.54mm_Vertical -> Connector_PinHeader_2.54mm:PinHeader_1x05_P2.54mm_Vertical
- U1: value AMS1117-3.3 -> XC6206PxxxMR; footprint Package_TO_SOT_SMD:SOT-223-3_TabPin2 -> Package_TO_SOT_SMD:SOT-23
- U2: value STM32F401RCTx -> STM32F411CCUx; footprint Package_QFP:LQFP-64_10x10mm_P0.5mm -> Package_DFN_QFN:QFN-48-1EP_7x7mm_P0.5mm_EP5.6x5.6mm
- moved SW1 78.4 mm to (190.5, 74.2)
- moved R1 62.1 mm to (176.3, 83.8)
- moved FB1 55.2 mm to (148.3, 90.2), turned to 90 degrees
- moved C10 52.4 mm to (146.5, 89.9), turned to 180 degrees
- moved C9 52.3 mm to (145.0, 91.7)
- moved C14 50.6 mm to (141.5, 87.7), turned to 180 degrees
- moved C3 50.5 mm to (190.5, 69.8), turned to 180 degrees
- moved C13 48.6 mm to (141.5, 84.6), turned to 180 degrees
- moved Y2 46.7 mm to (144.3, 86.1), turned to 90 degrees
- moved C12 37.6 mm to (142.7, 95.2), turned to 180 degrees
- moved Y1 35.6 mm to (140.7, 98.6)
- moved C11 34.6 mm to (138.7, 95.2)
- moved C4 31.4 mm to (153.2, 77.5), turned to -45 degrees
- moved C5 23.5 mm to (146.6, 81.8), turned to 45 degrees
- moved C6 23.2 mm to (157.5, 84.6), turned to -135 degrees
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Connections:
- net /STM32F401/PA5 renamed /STM32F411/PB10
- net /STM32F401/PB1 renamed /STM32F411/PBu14
- net /STM32F401/PB10 renamed /STM32F411/PA8
- net /STM32F401/PC13 renamed /STM32F411/PC13
- net /STM32F401/PC7 renamed /STM32F411/PA15
- net /STM32F401/VBAT_{I} renamed /STM32F411/VBAT_{I}
- net /STM32F401/XTAL_32K_1 renamed /STM32F411/XTAL_32K_1
- net /STM32F401/XTAL_32K_2 renamed /STM32F411/XTAL_32K_2
- net /STM32F401/XTAL_8M_1 renamed /STM32F411/XTAL_8M_1
- net /STM32F401/XTAL_8M_2 renamed /STM32F411/XTAL_8M_2
- C10 pad 1: /STM32F401/VREF+ -> /STM32F411/VREF+
- C101 pad 2: /USB_GND -> GND
- C102 pad 2: /USB_GND -> GND
- C3 pad 1: +3V3 -> /~{RST}
- C9 pad 1: /STM32F401/VREF+ -> /STM32F411/VREF+
- FB1 pad 2: /STM32F401/VREF+ -> /STM32F411/VREF+
- J102 pad 3: /USB_GND -> GND
- J103 pad 3: /STM32F401/PC1 -> /STM32F411/PB7
- J103 pad 5: /STM32F401/PC2 -> /STM32F411/PB6
- J103 pad 6: /STM32F401/PC5 -> /STM32F411/PB3
- J103 pad 7: /STM32F401/PC3 -> /STM32F411/PB5
- J103 pad 8: /STM32F401/PC4 -> /STM32F411/PB4
- J2 pad 2: /STM32F401/PA15 -> /STM32F411/PA13
- J2 pad 3: /~{RST} -> /STM32F411/PA14
- J2 pad 4: /STM32F401/PA13 -> /~{RST}
- J2 pad 5: /STM32F401/PB4 -> GND
- Q101 pad 1: /STM32F401/PA2 -> /STM32F411/PA2
- Q101 pad 3: /STM32F401/PA3 -> /STM32F411/PA3
- Q102 pad 2: /PB15 -> /STM32F411/PBu15
- R103 pad 2: /PB15 -> /STM32F411/PBu15
- R105 pad 2: /USB_GND -> GND
- R106 pad 1: /STM32F401/PA11 -> /STM32F411/PA11
- R107 pad 1: /STM32F401/PA12 -> /STM32F411/PA12
- R2 pad 1: /STM32F401/BOOT0 -> /STM32F411/BOOT0
- R3 pad 2: /STM32F401/PB2 -> /STM32F411/PB2
- SW101 pad 2: /STM32F401/PA1 -> /STM32F411/PA1
- SW102 pad 2: /STM32F401/PA0 -> /STM32F411/PA0
- U101 pad 1: /PB13 -> /STM32F411/PBu13
- U101 pad 5: /PB12 -> /STM32F411/PBu12
- U2 pad 10: /STM32F401/PC2 -> /STM32F411/PA0
- U2 pad 11: /STM32F401/PC3 -> /STM32F411/PA1
- U2 pad 12: GND -> /STM32F411/PA2
- U2 pad 13: /STM32F401/VREF+ -> /STM32F411/PA3
- U2 pad 14: /STM32F401/PA0 -> /STM32F411/PA4
- U2 pad 15: /STM32F401/PA1 -> /STM32F411/PA5
- U2 pad 16: /STM32F401/PA2 -> /STM32F411/PA6
- U2 pad 17: /STM32F401/PA3 -> /STM32F411/PA7
- U2 pad 18: GND -> /STM32F411/PB0
- U2 pad 19: +3V3 -> /STM32F411/PB1
- U2 pad 20: /STM32F401/PA4 -> /STM32F411/PB2
- U2 pad 22: /STM32F401/PA6 -> Net-(C8-Pad1)
- U2 pad 23: /STM32F401/PA7 -> GND
- U2 pad 24: /STM32F401/PC4 -> +3V3
- U2 pad 25: /STM32F401/PC5 -> /STM32F411/PBu12
- U2 pad 26: /STM32F401/PB0 -> /STM32F411/PBu13
- U2 pad 28: /STM32F401/PB2 -> /STM32F411/PBu15
- U2 pad 30: Net-(C8-Pad1) -> /STM32F411/PA9
- U2 pad 31: GND -> /STM32F411/PA10
- U2 pad 32: +3V3 -> /STM32F411/PA11
- U2 pad 33: /STM32F401/PB12 -> /STM32F411/PA12
- U2 pad 34: /STM32F401/PB13 -> /STM32F411/PA13
- U2 pad 35: /STM32F401/PB14 -> GND
- U2 pad 36: /STM32F401/PB15 -> +3V3
- U2 pad 37: /STM32F401/PC6 -> /STM32F411/PA14
- U2 pad 39: /STM32F401/PC8 -> /STM32F411/PB3
- U2 pad 40: /STM32F401/PC9 -> /STM32F411/PB4
- U2 pad 41: /STM32F401/PA8 -> /STM32F411/PB5
- U2 pad 42: /STM32F401/PA9 -> /STM32F411/PB6
- U2 pad 43: /STM32F401/PA10 -> /STM32F411/PB7
- U2 pad 44: /STM32F401/PA11 -> /STM32F411/BOOT0
- U2 pad 45: /STM32F401/PA12 -> /STM32F411/PB8
- U2 pad 46: /STM32F401/PA13 -> /STM32F411/PB9
- U2 pad 49: /STM32F401/PA14 -> GND
- U2 pad 8: /STM32F401/PC0 -> GND
- U2 pad 9: /STM32F401/PC1 -> /STM32F411/VREF+
Routing:
- net +3V3: track 1.27 -> 150.9 mm, vias 0 -> 7
- net /~{RST}: track 0.00 -> 125.7 mm, vias 0 -> 4
- net VCC: track 0.00 -> 123.5 mm, vias 0 -> 4
- net /STM32F411/PA3: track 0.00 -> 73.9 mm, vias 0 -> 2
- net /STM32F411/PA2: track 0.00 -> 69.8 mm, vias 0 -> 2
- net /STM32F411/PB3: track 0.00 -> 62.7 mm, vias 0 -> 2
- net /STM32F411/PB4: track 0.00 -> 56.1 mm, vias 0 -> 2
- net /STM32F411/PA1: track 0.00 -> 54.5 mm, vias 0 -> 1
- net /STM32F411/PBu12: track 0.00 -> 54.1 mm, vias 0 -> 4
- net /STM32F411/PA0: track 0.00 -> 53.9 mm, vias 0 -> 2
- net /STM32F411/PB7: track 0.00 -> 52.2 mm, vias 0 -> 2
- net /STM32F411/PB6: track 0.00 -> 51.3 mm, vias 0 -> 2
- net /STM32F411/PB5: track 0.00 -> 51.2 mm, vias 0 -> 2
- net /STM32F411/PBu13: track 0.00 -> 42.6 mm, vias 0 -> 2
- net /STM32F411/PBu15: track 0.00 -> 40.3 mm, vias 0 -> 2
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
Commit message: Finalize PCB
Other:
- board text added: "Frankenball Orbit v1 2022-06-18 GitHub: @CRTified"
